Commit message: fix a urdf file bug

File: 3.Software/Urdf_ConfigFiles/urdf/Urdf_ConfigFiles.urdf (robot description, URDF)
Before this commit: robot Urdf_ConfigFiles, 37 links, 35 joints
Joints:
- added joint LM_JIAN_JOINT: type revolute, parent base_link, child LM_JIAN_LINK, origin xyz=0 0.050828 0.0047 rpy=0 0 1.5708, axis 0 0 1, limit lower=-1.5708 upper=1.5708 effort=0 velocity=0
- joint LF_JIAN_JOINT: child LM_JIAN_LINK -> LF_JIAN_LINK; origin xyz=0 0.050828 0.0047 rpy=0 0 1.5708 -> xyz=0.077746 0.036979 0.0047 rpy=0 0 0.7854

Commit message: update kinetic source code

File: 3.Software/Urdf_ConfigFiles/urdf/Urdf_ConfigFiles.urdf (robot description, URDF)
Before this commit: robot Urdf_ConfigFiles, 37 links, 36 joints
Joints:
- removed joint LM_P_JOIINT
- removed joint RF_P_LINK
- added joint LM_P_JOINT: type revolute, parent LM_R_LINK, child LM_P_LINK, origin xyz=0 0 0 rpy=0 1.5708 0, axis 0 0 -1, limit lower=-1.5708 upper=1.5708 effort=0 velocity=0
- added joint RF_P_JOINT: type revolute, parent RF_R_LINK, child RF_P_LINK, origin xyz=0 0 0 rpy=0 1.5708 0, axis 0 0 1, limit lower=-1.5708 upper=1.5708 effort=0 velocity=0
